Commit message: controllers works, but pid values and effort limits of joints are not correct. Maybe also world settings of friction values needs to be tuned

File: urdf/handy_robot_gazebo.urdf (robot description, URDF)
Before this commit: robot handy robot gazebo, 7 links, 6 joints
Joints:
- joint elbow_joint: limit lower=0 upper=3.14 effort=0.1 velocity=0.005 -> lower=0 upper=3.14 effort=1 velocity=0.005
- joint slider_joint: limit lower=0 upper=0.3 effort=0.1 velocity=0.005 -> lower=0 upper=0.3 effort=1 velocity=0.005
